File: GY-PCM5102A.kicad_sch (KiCad schematic)
At the start: 30 parts, among them J1 M-BUS, J2 FUN_AND_OUT, J3 AudioJack3, U1 PCM5102A, U2 ME6211C33M5, U3 ME6211C33M5

Commit message: feat: populate PCB and update schematic
Parts:
- C10, C7, C8, C9: footprint (none) -> Capacitor_SMD:C_0603_1608Metric
- C11, C13: footprint Capacitor_Tantalum_SMD:CP_EIA-3528-21_Kemet-B -> Capacitor_SMD:C_0603_1608Metric; symbol Device:C_Polarized -> Device:C
- C3, C5: footprint Capacitor_Tantalum_SMD:CP_EIA-3528-21_Kemet-B -> Capacitor_SMD:C_0805_2012Metric; symbol Device:C_Polarized -> Device:C
- FP1: renamed from H1L; footprint Jumper:SolderJumper-3_P1.3mm_Open_Pad1.0x1.5mm -> Jumper_custom:SolderJumper-3_P1.3mm_Open_Pad0.55x1.15mm
- FP2: renamed from H2L; footprint Jumper:SolderJumper-3_P1.3mm_Open_Pad1.0x1.5mm -> Jumper_custom:SolderJumper-3_P1.3mm_Open_Pad0.55x1.15mm
- FP3: renamed from H3L; footprint Jumper:SolderJumper-3_P1.3mm_Open_Pad1.0x1.5mm -> Jumper_custom:SolderJumper-3_P1.3mm_Open_Pad0.55x1.15mm
- FP4: renamed from H4L; footprint Jumper:SolderJumper-3_P1.3mm_Open_Pad1.0x1.5mm -> Jumper_custom:SolderJumper-3_P1.3mm_Open_Pad0.55x1.15mm
- J2: footprint (none) -> Connector_PinHeader_2.54mm:PinHeader_1x09_P2.54mm_Vertical
Connections:
- net GND: now also C10.2, C7.2, C9.2; no longer C10.1, C7.1, C9.1
- net OUTL: now also C9.1, J3.T, R2.2; no longer R2.1, U1.6 (OUTL)
- net OUTR: now also C10.1, J3.R, R3.2; no longer R3.1, U1.7 (OUTR)
- net at U1.2 (CAPP): now also C8.1; no longer C8.2
- net at U1.4 (CAPM): now also C8.2; no longer C8.1
- net at U1.5 (VNEG): now also C7.1; no longer C7.2
- new net: R3.1, U1.7 (OUTR)
- new net: R2.1, U1.6 (OUTL)
